Commit message: updating all files hawl

File: roscourse_sim_ws/install/my_robot/share/my_robot/my_robot.urdf.xacro (robot description, xacro)
@@ -151,3 +151,27 @@
         <origin xyz="0 0 0.1" rpy="0 0 0" />
     </joint>
+    <gazebo reference="base_link">
+        <material>Gazebo/Green</material>
+    </gazebo>
+    <gazebo>
+        <plugin name="diff_drive_controller" filename="libgazebo_ros_diff_drive.so">
+        <!-- Update rate in Hz -->
+        <update_rate>50</update_rate>
+        <!-- wheels -->
+        <left_joint>base_left_wheel_joint</left_joint>
+        <right_joint>base_right_wheel_joint</right_joint>
+        <!-- kinematics -->
+        <wheel_separation>0.4</wheel_separation>
+        <wheel_diameter>0.2</wheel_diameter>
+        <!-- output -->
+        <publish_odom>true</publish_odom>
+        <publish_odom_tf>true</publish_odom_tf>
+        <publish_wheel_tf>true</publish_wheel_tf>
+        <odometry_topic>odom</odometry_topic>
+        <odometry_frame>odom</odometry_frame>
+        <robot_base_frame>base_footprint</robot_base_frame>
+        <!-- input -->
+        <command_topic>cmd_vel</command_topic>
+        </plugin>
+    </gazebo>
 </robot>
