Commit message: Added collision geometry, meshes still not showing

File: project_ws/src/rosmaster_sim/urdf/yahboomcar_X3.urdf (robot description, URDF)
Before this commit: robot yahboomcar, 9 links, 8 joints
Links:
- link base_link: geometry collision box size=0.5 0.5 0.5; visual mesh filename=package://rosmaster_sim/meshes/mecanum/base_link.STL
Joints:
- joint back_left_joint: type continuous -> fixed
- joint back_right_joint: type continuous -> fixed
- joint front_left_joint: type continuous -> fixed
- joint front_right_joint: type continuous -> fixed

Commit message: Testing sending shape coords

File: project_ws/src/rosmaster_sim/urdf/yahboomcar_X3.urdf (robot description, URDF)
Before this commit: robot yahboomcar, 9 links, 8 joints
Links:
- link base_link: geometry collision box size=0.5 0.5 0.3; visual mesh filename=package://rosmaster_sim/meshes/mecanum/base_link.STL
- link front_left_wheel: geometry collision mesh filename=package://rosmaster_sim/meshes/mecanum/front_left_wheel.STL; visual mesh filename=${find rosmaster_sim/meshes/mecanum/front_left_wheel.STL}
